File: nucleo_144_hat.kicad_pcb (KiCad board)
At the start: 4 copper layers, 71.5 x 101.5 mm, 23 parts, among them J1 SPI1_Conn_01x07, J10 CAN2_OUT_Conn_01x04, J11 CAN1_OUT_Conn_01x04, J12 Conn_01x02, J2 PWM_OUT_Conn_01x06, J3 ADC1_Conn_01x04, J4 UART1_Conn_01x06, J5 UART2_Conn_01x06, J6 UART3_Conn_01x06, J7 UART4_Conn_01x06, J8 CAN1_IN_Conn_01x04, J9 CAN2_IN_Conn_01x04, U1 NUCLEO144-F767ZI, U2 TJA1051TK-3, U3 TJA1051TK-3

Commit message: clean up tracing
Parts:
- J10: value CAN2_OUT_Conn_01x04 -> CAN2_B_Conn_01x04
- J11: value CAN1_OUT_Conn_01x04 -> CAN1_B_Conn_01x04
- J8: value CAN1_IN_Conn_01x04 -> CAN1_A_Conn_01x04
- J9: value CAN2_IN_Conn_01x04 -> CAN2_A_Conn_01x04
Routing:
- net +3V3: track 138.2 -> 8.17 mm
- net /~{SPI2_CS2}: track 57.7 -> 70.2 mm
- net /UART2_RTS: track 55.0 -> 65.4 mm
- net /UART2_CTS: track 50.9 -> 60.9 mm
- net /UART3_TX: track 81.4 -> 74.3 mm
- net /SPI1_SCK: track 54.4 -> 60.1 mm
- net /SPI1_MISO: track 52.2 -> 56.8 mm
- net /CAN1_TX: track 34.0 -> 37.9 mm
- net /UART4_CTS: track 62.2 -> 59.5 mm
- net /UART1_TX: track 19.6 -> 21.4 mm
- net /UART4_TX: track 29.2 -> 30.9 mm
- net /UART1_RTS: track 17.1 -> 18.6 mm
- net /UART4_RX: track 26.4 -> 25.4 mm
- net /CAN2_RX: track 63.9 -> 64.8 mm
- net /CAN2_TX: track 77.0 -> 77.7 mm
- added copper zone on B.Cu, net +3V3
