File: nucleo_144_hat.kicad_sch (KiCad schematic)
At the start: 23 parts, among them J1 SPI1_Conn_01x07, J10 CAN2_OUT_Conn_01x04, J11 CAN1_OUT_Conn_01x04, J12 Conn_01x02, J2 PWM_OUT_Conn_01x06, J3 ADC1_Conn_01x04, J4 UART1_Conn_01x06, J5 UART2_Conn_01x06, J6 UART3_Conn_01x06, J7 UART4_Conn_01x06, J8 CAN1_IN_Conn_01x04, J9 CAN2_IN_Conn_01x04, U1 NUCLEO144-F767ZI, U2 TJA1051TK-3, U3 TJA1051TK-3

Commit message: clean up tracing
Parts:
- J10: value CAN2_OUT_Conn_01x04 -> CAN2_B_Conn_01x04
- J11: value CAN1_OUT_Conn_01x04 -> CAN1_B_Conn_01x04
- J8: value CAN1_IN_Conn_01x04 -> CAN1_A_Conn_01x04
- J9: value CAN2_IN_Conn_01x04 -> CAN2_A_Conn_01x04
Changed lines of the file:
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@@
       (effects (font (size 1.27 1.27)) (justify left))
     )
-    (property "Value" "CAN2_IN_Conn_01x04" (id 1) (at 281.94 91.4399 0)
+    (property "Value" "CAN2_A_Conn_01x04" (id 1) (at 281.94 91.4399 0)
       (effects (font (size 1.27 1.27)) (justify left))
     )
@@
       (effects (font (size 1.27 1.27)) (justify left))
     )
-    (property "Value" "CAN2_OUT_Conn_01x04" (id 1) (at 281.94 107.3149 0)
+    (property "Value" "CAN2_B_Conn_01x04" (id 1) (at 281.94 107.3149 0)
       (effects (font (size 1.27 1.27)) (justify left))
     )
@@
       (effects (font (size 1.27 1.27)) (justify left))
     )
-    (property "Value" "CAN1_IN_Conn_01x04" (id 1) (at 281.94 55.8799 0)
+    (property "Value" "CAN1_A_Conn_01x04" (id 1) (at 281.94 55.8799 0)
       (effects (font (size 1.27 1.27)) (justify left))
     )
@@
   (symbol (lib_id "Connector_Generic:Conn_01x04") (at 280.035 68.58 0) (unit 1)
     (in_bom yes) (on_board yes) (fields_autoplaced)
-    (property "Reference" "J11" (id 0) (at 282.575 68.5799 0)
-      (effects (font (size 1.27 1.27)) (justify left))
-    )
-    (property "Value" "CAN1_OUT_Conn_01x04" (id 1) (at 282.575 71.1199 0)
+    (property "Reference" "J11" (id 0) (at 283.21 68.5799 0)
+      (effects (font (size 1.27 1.27)) (justify left))
+    )
+    (property "Value" "CAN1_B_Conn_01x04" (id 1) (at 283.21 71.1199 0)
       (effects (font (size 1.27 1.27)) (justify left))
     )
@@
     )
     (path "/79822b91-c2ca-44d1-b161-fb2c7fc4c3e3"
-      (reference "J8") (unit 1) (value "CAN1_IN_Conn_01x04") (footprint "Connector_JST:JST_GH_SM04B-GHS-TB_1x04-1MP_P1.25mm_Horizontal")
+      (reference "J8") (unit 1) (value "CAN1_A_Conn_01x04") (footprint "Connector_JST:JST_GH_SM04B-GHS-TB_1x04-1MP_P1.25mm_Horizontal")
     )
     (path "/08501816-c00a-45cf-a10a-1ed7cf05624e"
-      (reference "J9") (unit 1) (value "CAN2_IN_Conn_01x04") (footprint "Connector_JST:JST_GH_SM04B-GHS-TB_1x04-1MP_P1.25mm_Horizontal")
+      (reference "J9") (unit 1) (value "CAN2_A_Conn_01x04") (footprint "Connector_JST:JST_GH_SM04B-GHS-TB_1x04-1MP_P1.25mm_Horizontal")
     )
     (path "/12c05adb-b4a5-4dbc-89a5-65704a123684"
-      (reference "J10") (unit 1) (value "CAN2_OUT_Conn_01x04") (footprint "Connector_JST:JST_GH_SM04B-GHS-TB_1x04-1MP_P1.25mm_Horizontal")
+      (reference "J10") (unit 1) (value "CAN2_B_Conn_01x04") (footprint "Connector_JST:JST_GH_SM04B-GHS-TB_1x04-1MP_P1.25mm_Horizontal")
     )
     (path "/a4582c70-e32c-4e85-bab1-bb2f99742d91"
-      (reference "J11") (unit 1) (value "CAN1_OUT_Conn_01x04") (footprint "Connector_JST:JST_GH_SM04B-GHS-TB_1x04-1MP_P1.25mm_Horizontal")
+      (reference "J11") (unit 1) (value "CAN1_B_Conn_01x04") (footprint "Connector_JST:JST_GH_SM04B-GHS-TB_1x04-1MP_P1.25mm_Horizontal")
     )
     (path "/0fbaa32d-2728-4518-ae79-7fc37cbde580"
